Commit message: Bug fixing on config files

File: urdf/ur10e_eecam.xacro (robot description, xacro)
@@ -19,11 +19,11 @@
   <!-- Fixed joint camera -->
   <joint name="camera_robot_joint" type="fixed">
-    <origin xyz="0.1 0.1 0.1" rpy="0 0 0"/>
+    <origin xyz="0.1 0.1 0.1" rpy="0 -1.570796327 1.570796327"/>
     <parent link="tool0"/>
-    <child link="camera_base_link"/>
+    <child  link="camera_base_link"/>
   </joint>
   <!-- Import d435 xacro file -->
   <xacro:include filename="$(find realsense2_description)/urdf/_d435.urdf.xacro" />
-  <link name="camera_base_link" />
+  <link name="camera_base_link"/>
   <xacro:sensor_d435 parent="camera_base_link" use_nominal_extrinsics="false" add_plug="false" use_mesh="true">
     <origin xyz="0 0 0" rpy="0 0 0"/>

Commit message: Added launch args to ur10eecam xacro file, now starting position of camera can be changed from the ur10 planner launch

File: urdf/ur10e_eecam.xacro (robot description, xacro)
@@ -1,17 +1,12 @@
 <?xml version="1.0"?>
 <robot xmlns:xacro="http://wiki.ros.org/xacro" name="ur10e_robot">
-  <!--
-    This is a convenience top-level xacro which loads the macro for the UR10e
-    which defines the default values for the various "parameters files"
-    parameters for a UR10e.
-    This file is only useful when loading a stand-alone, completely isolated
-    robot with only default values for all parameters such as the kinematics,
-    visual and physical parameters and joint limits.
-    This file is not intended to be integrated into a larger scene or other
-    composite xacro.
-    Instead, xacro:include 'inc/ur10e_macro.xacro' and override the defaults
-    for the arguments to that macro.
-    Refer to 'inc/ur_macro.xacro' for more information.
-  -->
+  <!-- Args for starting camera position -->
+  <xacro:arg name="cam_x_offset"  default="+0.1"/>
+  <xacro:arg name="cam_y_offset"  default="+0.1"/>
+  <xacro:arg name="cam_z_offset"  default="+0.1"/>
+  <xacro:arg name="cam_rx"        default="+0.0"/>
+  <xacro:arg name="cam_ry"        default="-1.570796327"/>
+  <xacro:arg name="cam_rz"        default="-1.570796327"/>
+  <xacro:arg name="cam_parent"    default="tool0"/>
   <!-- Import robot ur10 xacro file -->
   <xacro:include filename="$(find ur_description)/urdf/inc/ur10e_macro.xacro"/>
@@ -19,6 +14,7 @@
   <!-- Fixed joint camera -->
   <joint name="camera_robot_joint" type="fixed">
-    <origin xyz="0.1 0.1 0.1" rpy="0 -1.570796327 1.570796327"/>
-    <parent link="tool0"/>
+    <origin xyz="$(arg cam_x_offset) $(arg cam_y_offset) $(arg cam_z_offset)"
+            rpy="$(arg cam_rx) $(arg cam_ry) $(arg cam_rz)"/>
+    <parent link="$(arg cam_parent)"/>
     <child  link="camera_base_link"/>
   </joint>

Commit message: Group ur10+camera+gripper perfectly working

File: urdf/ur10e_eecam.xacro (robot description, xacro)
@@ -9,4 +9,8 @@
   <xacro:arg name="cam_rz"        default="-1.570796327"/>
   <xacro:arg name="cam_parent"    default="tool0"/>
+  <!-- Args for starting gripper position -->
+  <xacro:arg name="ee_z_offset"   default="+0.0"/>
+  <xacro:arg name="ee_rz"         default="+0.0"/>
+  <xacro:arg name="ee_parent"     default="tool0"/>
   <!-- Import robot ur10 xacro file -->
   <xacro:include filename="$(find ur_description)/urdf/inc/ur10e_macro.xacro"/>
@@ -25,3 +29,11 @@
     <origin xyz="0 0 0" rpy="0 0 0"/>
   </xacro:sensor_d435>
+  <!-- Import Robotiq85Gripper -->
+  <xacro:include filename="$(find robotiq85_gripper)/models/robotiq_85.URDF"/>
+  <!-- Fixed joint gripper -->
+  <joint name="gripper_robot_joint" type="fixed">
+    <origin xyz="0 0 $(arg ee_z_offset)" rpy="0 0 $(arg ee_rz)"/>
+    <parent link="$(arg ee_parent)"/>
+    <child  link="robotiq_85_base_link"/>
+  </joint>
 </robot>
