Commit message: Modified planning launch interface; now future grippers and cameras can be easily integrated in robots urdf description and planning scene without issues, warning, errors and illogic sequential actions

File: models/urdf/ur10e_eecam.xacro (robot description, xacro)
@@ -27,5 +27,12 @@
   <!-- Import d435 xacro file -->
   <xacro:include filename="$(find realsense2_description)/urdf/_d435.urdf.xacro" />
-  <link name="camera_base_link"/>
+  <link name="camera_base_link">
+  <collision>
+    <origin xyz="-0.0061 0.0 +0.0125" rpy="0 0 0"/>
+    <geometry>
+      <box size="0.0083 0.09 0.025"/>
+    </geometry>
+  </collision>
+  </link>
   <xacro:sensor_d435 parent="camera_base_link" use_nominal_extrinsics="false" add_plug="false" use_mesh="true">
     <origin xyz="0 0 0" rpy="0 0 0"/>

Commit message: Uploaded urdf file of ur10e with ee and camera

File: models/urdf/ur10e_eecam.xacro (robot description, xacro)
@@ -1,18 +1,18 @@
 <?xml version="1.0"?>
 <!-- To convert to urdf use the command:
-     rosrun xacro xacro (minus)(minus)inorder -o model.urdf model.urdf.xacro -->
+     rosrun xacro xacro -o model.urdf model.urdf.xacro -->
 <robot xmlns:xacro="http://wiki.ros.org/xacro" name="ur10e_eecam_robot">
   <!-- Args for starting camera position -->
-  <xacro:arg name="cam_x_offset"  default="+0.1"/>
-  <xacro:arg name="cam_y_offset"  default="+0.1"/>
-  <xacro:arg name="cam_z_offset"  default="+0.1"/>
+  <xacro:arg name="cam_parent"    default="tool0"/>
+  <xacro:arg name="cam_x_offset"  default="+0.0"/>
+  <xacro:arg name="cam_y_offset"  default="+0.05"/>
+  <xacro:arg name="cam_z_offset"  default="+0.05"/>
   <xacro:arg name="cam_rx"        default="+0.0"/>
   <xacro:arg name="cam_ry"        default="-1.570796327"/>
   <xacro:arg name="cam_rz"        default="-1.570796327"/>
-  <xacro:arg name="cam_parent"    default="tool0"/>
   <!-- Args for starting gripper position -->
+  <xacro:arg name="ee_parent"     default="tool0"/>
   <xacro:arg name="ee_z_offset"   default="+0.0"/>
   <xacro:arg name="ee_rz"         default="+0.0"/>
-  <xacro:arg name="ee_parent"     default="tool0"/>
   <!-- Import robot ur10 xacro file -->
   <xacro:include filename="$(find ur_description)/urdf/inc/ur10e_macro.xacro"/>
@@ -28,10 +28,10 @@
   <xacro:include filename="$(find realsense2_description)/urdf/_d435.urdf.xacro" />
   <link name="camera_base_link">
-  <collision>
-    <origin xyz="-0.0061 0.0 +0.0125" rpy="0 0 0"/>
-    <geometry>
-      <box size="0.0083 0.09 0.025"/>
-    </geometry>
-  </collision>
+    <collision>
+      <origin xyz="-0.0061 0.0 +0.0125" rpy="0 0 0"/>
+      <geometry>
+        <box size="0.0083 0.09 0.025"/>
+      </geometry>
+    </collision>
   </link>
   <xacro:sensor_d435 parent="camera_base_link" use_nominal_extrinsics="false" add_plug="false" use_mesh="true">

Commit message: Added tcp link-joint to ur10e_eecam model

File: models/urdf/ur10e_eecam.xacro (robot description, xacro)
@@ -15,4 +15,5 @@
   <xacro:arg name="ee_z_offset"   default="+0.0"/>
   <xacro:arg name="ee_rz"         default="+0.0"/>
+  <xacro:arg name="tcp_offset"    default="+0.122"/>
   <!-- Import robot ur10 xacro file -->
   <xacro:include filename="$(find ur_description)/urdf/inc/ur10e_macro.xacro"/>
@@ -46,3 +47,10 @@
     <child  link="robotiq_85_base_link"/>
   </joint>
+  <!-- Fixed tcp gripper -->
+  <link name="tcp_gripper"/>
+  <joint name="tcp_gripper_joint" type="fixed">
+    <origin xyz="0 0 $(arg tcp_offset)" rpy="0 0 0"/>
+    <parent link="robotiq_85_base_link"/>
+    <child  link="tcp_gripper"/>
+  </joint>
 </robot>
