Commit message: Universal robot planner completed. All functions generalized for all urs

File: models/urdf/ur10.xacro (robot description, xacro)
@@ -1,8 +1,8 @@
 <?xml version="1.0"?>
-<robot xmlns:xacro="http://wiki.ros.org/xacro" name="ur3_robot">
+<robot xmlns:xacro="http://wiki.ros.org/xacro" name="ur10_robot">
   <!--
-    This is a convenience top-level xacro which loads the macro for the UR3
+    This is a convenience top-level xacro which loads the macro for the UR10
     which defines the default values for the various "parameters files"
-    parameters for a UR3.
+    parameters for a UR10.
     This file is only useful when loading a stand-alone, completely isolated
     robot with only default values for all parameters such as the kinematics,
@@ -10,5 +10,5 @@
     This file is not intended to be integrated into a larger scene or other
     composite xacro.
-    Instead, xacro:include 'inc/ur3_macro.xacro' and override the defaults
+    Instead, xacro:include 'inc/ur10_macro.xacro' and override the defaults
     for the arguments to that macro.
     Refer to 'inc/ur_macro.xacro' for more information.
@@ -30,7 +30,7 @@
   <xacro:arg name="ee_rz"         default="+0.00"/>
   <xacro:arg name="tcp_offset"    default="+0.00"/>
-  <!-- Include ur3 model -->
-  <xacro:include filename="$(find ur_description)/urdf/inc/ur3_macro.xacro"/>
-  <xacro:ur3_robot prefix="" />
+  <!-- Include ur10 model -->
+  <xacro:include filename="$(find ur_description)/urdf/inc/ur10_macro.xacro"/>
+  <xacro:ur10_robot prefix="" />
   <!-- Fixed tcp gripper -->
   <link name="tcp_gripper"/>

File: models/urdf/ur10e.xacro (robot description, xacro)
@@ -16,16 +16,18 @@
   <!-- Args for starting ee tool position -->
     <!-- Args for starting camera position -->
+  <xacro:arg name="camera"        default="false"/>
   <xacro:arg name="cam_parent"    default="tool0"/>
-  <xacro:arg name="cam_x_offset"  default="+0.0"/>
-  <xacro:arg name="cam_y_offset"  default="+0.05"/>
-  <xacro:arg name="cam_z_offset"  default="+0.05"/>
-  <xacro:arg name="cam_rx"        default="+0.0"/>
+  <xacro:arg name="cam_x_offset"  default="+0.00"/>
+  <xacro:arg name="cam_y_offset"  default="+0.00"/>
+  <xacro:arg name="cam_z_offset"  default="+0.00"/>
+  <xacro:arg name="cam_rx"        default="+0.00"/>
   <xacro:arg name="cam_ry"        default="-1.570796327"/>
   <xacro:arg name="cam_rz"        default="-1.570796327"/>
   <!-- Args for starting gripper position -->
+  <xacro:arg name="ee"            default="false"/>
   <xacro:arg name="ee_parent"     default="tool0"/>
-  <xacro:arg name="ee_z_offset"   default="+0.0"/>
-  <xacro:arg name="ee_rz"         default="+0.0"/>
-  <xacro:arg name="tcp_offset"    default="+0.05"/>
+  <xacro:arg name="ee_z_offset"   default="+0.00"/>
+  <xacro:arg name="ee_rz"         default="+0.00"/>
+  <xacro:arg name="tcp_offset"    default="+0.00"/>
   <!-- Include ur10e model -->
   <xacro:include filename="$(find ur_description)/urdf/inc/ur10e_macro.xacro"/>
@@ -35,6 +37,40 @@
   <joint name="tcp_gripper_joint" type="fixed">
     <origin xyz="0 0 $(arg tcp_offset)" rpy="0 0 0"/>
-    <parent link="$(arg ee_parent)"/>
+    <parent link="tool0"/>
     <child  link="tcp_gripper"/>
   </joint>
+  <!-- Add camera -->
+  <xacro:if value="$(arg camera)">
+    <!-- Fixed joint camera -->
+    <joint name="camera_robot_joint" type="fixed">
+      <origin xyz="$(arg cam_x_offset) $(arg cam_y_offset) $(arg cam_z_offset)"
+              rpy="$(arg cam_rx) $(arg cam_ry) $(arg cam_rz)"/>
+      <parent link="$(arg cam_parent)"/>
+      <child  link="camera_base_link"/>
+    </joint>
+    <!-- Import d435 xacro file -->
+    <xacro:include filename="$(find realsense2_description)/urdf/_d435.urdf.xacro" />
+    <link name="camera_base_link">
+      <collision>
+        <origin xyz="-0.0061 0.0 +0.0125" rpy="0 0 0"/>
+        <geometry>
+          <box size="0.0083 0.09 0.025"/>
+        </geometry>
+      </collision>
+    </link>
+    <xacro:sensor_d435 parent="camera_base_link" use_nominal_extrinsics="false" add_plug="false" use_mesh="true">
+      <origin xyz="0 0 0" rpy="0 0 0"/>
+    </xacro:sensor_d435>
+  </xacro:if>
+  <!-- Add end-effector -->
+  <xacro:if value="$(arg ee)">
+    <!-- Import Robotiq85Gripper -->
+    <xacro:include filename="$(find gripper)/models/robotiq_85.urdf.xacro"/>
+    <!-- Fixed joint gripper -->
+    <joint name="gripper_robot_joint" type="fixed">
+      <origin xyz="0 0 $(arg ee_z_offset)" rpy="0 0 $(arg ee_rz)"/>
+      <parent link="$(arg ee_parent)"/>
+      <child  link="robotiq_85_base_link"/>
+    </joint>
+  </xacro:if>
 </robot>

File: models/urdf/ur16e.xacro (robot description, xacro)
@@ -1,8 +1,8 @@
 <?xml version="1.0"?>
-<robot xmlns:xacro="http://wiki.ros.org/xacro" name="ur5e_robot">
+<robot xmlns:xacro="http://wiki.ros.org/xacro" name="ur16e_robot">
   <!--
-    This is a convenience top-level xacro which loads the macro for the UR10e
+    This is a convenience top-level xacro which loads the macro for the UR16e
     which defines the default values for the various "parameters files"
-    parameters for a UR5e.
+    parameters for a UR16e.
     This file is only useful when loading a stand-alone, completely isolated
     robot with only default values for all parameters such as the kinematics,
@@ -10,5 +10,5 @@
     This file is not intended to be integrated into a larger scene or other
     composite xacro.
-    Instead, xacro:include 'inc/ur5e_macro.xacro' and override the defaults
+    Instead, xacro:include 'inc/ur16e_macro.xacro' and override the defaults
     for the arguments to that macro.
     Refer to 'inc/ur_macro.xacro' for more information.
@@ -16,25 +16,61 @@
   <!-- Args for starting ee tool position -->
     <!-- Args for starting camera position -->
+  <xacro:arg name="camera"        default="false"/>
   <xacro:arg name="cam_parent"    default="tool0"/>
-  <xacro:arg name="cam_x_offset"  default="+0.0"/>
-  <xacro:arg name="cam_y_offset"  default="+0.05"/>
-  <xacro:arg name="cam_z_offset"  default="+0.05"/>
-  <xacro:arg name="cam_rx"        default="+0.0"/>
+  <xacro:arg name="cam_x_offset"  default="+0.00"/>
+  <xacro:arg name="cam_y_offset"  default="+0.00"/>
+  <xacro:arg name="cam_z_offset"  default="+0.00"/>
+  <xacro:arg name="cam_rx"        default="+0.00"/>
   <xacro:arg name="cam_ry"        default="-1.570796327"/>
   <xacro:arg name="cam_rz"        default="-1.570796327"/>
   <!-- Args for starting gripper position -->
+  <xacro:arg name="ee"            default="false"/>
   <xacro:arg name="ee_parent"     default="tool0"/>
-  <xacro:arg name="ee_z_offset"   default="+0.0"/>
-  <xacro:arg name="ee_rz"         default="+0.0"/>
-  <xacro:arg name="tcp_offset"    default="+0.05"/>
-  <!-- Include ur5e model -->
-  <xacro:include filename="$(find ur_description)/urdf/inc/ur5e_macro.xacro"/>
-  <xacro:ur5e_robot prefix="" />
+  <xacro:arg name="ee_z_offset"   default="+0.00"/>
+  <xacro:arg name="ee_rz"         default="+0.00"/>
+  <xacro:arg name="tcp_offset"    default="+0.00"/>
+  <!-- Include ur16e model -->
+  <xacro:include filename="$(find ur_description)/urdf/inc/ur16e_macro.xacro"/>
+  <xacro:ur16e_robot prefix="" />
   <!-- Fixed tcp gripper -->
   <link name="tcp_gripper"/>
   <joint name="tcp_gripper_joint" type="fixed">
     <origin xyz="0 0 $(arg tcp_offset)" rpy="0 0 0"/>
-    <parent link="$(arg ee_parent)"/>
+    <parent link="tool0"/>
     <child  link="tcp_gripper"/>
   </joint>
+  <!-- Add camera -->
+  <xacro:if value="$(arg camera)">
+    <!-- Fixed joint camera -->
+    <joint name="camera_robot_joint" type="fixed">
+      <origin xyz="$(arg cam_x_offset) $(arg cam_y_offset) $(arg cam_z_offset)"
+              rpy="$(arg cam_rx) $(arg cam_ry) $(arg cam_rz)"/>
+      <parent link="$(arg cam_parent)"/>
+      <child  link="camera_base_link"/>
+    </joint>
+    <!-- Import d435 xacro file -->
+    <xacro:include filename="$(find realsense2_description)/urdf/_d435.urdf.xacro" />
+    <link name="camera_base_link">
+      <collision>
+        <origin xyz="-0.0061 0.0 +0.0125" rpy="0 0 0"/>
+        <geometry>
+          <box size="0.0083 0.09 0.025"/>
+        </geometry>
+      </collision>
+    </link>
+    <xacro:sensor_d435 parent="camera_base_link" use_nominal_extrinsics="false" add_plug="false" use_mesh="true">
+      <origin xyz="0 0 0" rpy="0 0 0"/>
+    </xacro:sensor_d435>
+  </xacro:if>
+  <!-- Add end-effector -->
+  <xacro:if value="$(arg ee)">
+    <!-- Import Robotiq85Gripper -->
+    <xacro:include filename="$(find gripper)/models/robotiq_85.urdf.xacro"/>
+    <!-- Fixed joint gripper -->
+    <joint name="gripper_robot_joint" type="fixed">
+      <origin xyz="0 0 $(arg ee_z_offset)" rpy="0 0 $(arg ee_rz)"/>
+      <parent link="$(arg ee_parent)"/>
+      <child  link="robotiq_85_base_link"/>
+    </joint>
+  </xacro:if>
 </robot>

File: models/urdf/ur20.xacro (robot description, xacro)
@@ -1,8 +1,8 @@
 <?xml version="1.0"?>
-<robot xmlns:xacro="http://wiki.ros.org/xacro" name="ur3_robot">
+<robot xmlns:xacro="http://wiki.ros.org/xacro" name="ur20_robot">
   <!--
-    This is a convenience top-level xacro which loads the macro for the UR3
+    This is a convenience top-level xacro which loads the macro for the UR20
     which defines the default values for the various "parameters files"
-    parameters for a UR3.
+    parameters for a UR20.
     This file is only useful when loading a stand-alone, completely isolated
     robot with only default values for all parameters such as the kinematics,
@@ -10,5 +10,5 @@
     This file is not intended to be integrated into a larger scene or other
     composite xacro.
-    Instead, xacro:include 'inc/ur3_macro.xacro' and override the defaults
+    Instead, xacro:include 'inc/ur20_macro.xacro' and override the defaults
     for the arguments to that macro.
     Refer to 'inc/ur_macro.xacro' for more information.
@@ -30,7 +30,7 @@
   <xacro:arg name="ee_rz"         default="+0.00"/>
   <xacro:arg name="tcp_offset"    default="+0.00"/>
-  <!-- Include ur3 model -->
-  <xacro:include filename="$(find ur_description)/urdf/inc/ur3_macro.xacro"/>
-  <xacro:ur3_robot prefix="" />
+  <!-- Include ur20 model -->
+  <xacro:include filename="$(find ur_description)/urdf/inc/ur20_macro.xacro"/>
+  <xacro:ur20_robot prefix="" />
   <!-- Fixed tcp gripper -->
   <link name="tcp_gripper"/>

File: models/urdf/ur3e.xacro (robot description, xacro)
@@ -1,8 +1,8 @@
 <?xml version="1.0"?>
-<robot xmlns:xacro="http://wiki.ros.org/xacro" name="ur5e_robot">
+<robot xmlns:xacro="http://wiki.ros.org/xacro" name="ur3e_robot">
   <!--
-    This is a convenience top-level xacro which loads the macro for the UR10e
+    This is a convenience top-level xacro which loads the macro for the UR3e
     which defines the default values for the various "parameters files"
-    parameters for a UR5e.
+    parameters for a UR3e.
     This file is only useful when loading a stand-alone, completely isolated
     robot with only default values for all parameters such as the kinematics,
@@ -10,5 +10,5 @@
     This file is not intended to be integrated into a larger scene or other
     composite xacro.
-    Instead, xacro:include 'inc/ur5e_macro.xacro' and override the defaults
+    Instead, xacro:include 'inc/ur3e_macro.xacro' and override the defaults
     for the arguments to that macro.
     Refer to 'inc/ur_macro.xacro' for more information.
@@ -16,25 +16,61 @@
   <!-- Args for starting ee tool position -->
     <!-- Args for starting camera position -->
+  <xacro:arg name="camera"        default="false"/>
   <xacro:arg name="cam_parent"    default="tool0"/>
-  <xacro:arg name="cam_x_offset"  default="+0.0"/>
-  <xacro:arg name="cam_y_offset"  default="+0.05"/>
-  <xacro:arg name="cam_z_offset"  default="+0.05"/>
-  <xacro:arg name="cam_rx"        default="+0.0"/>
+  <xacro:arg name="cam_x_offset"  default="+0.00"/>
+  <xacro:arg name="cam_y_offset"  default="+0.00"/>
+  <xacro:arg name="cam_z_offset"  default="+0.00"/>
+  <xacro:arg name="cam_rx"        default="+0.00"/>
   <xacro:arg name="cam_ry"        default="-1.570796327"/>
   <xacro:arg name="cam_rz"        default="-1.570796327"/>
   <!-- Args for starting gripper position -->
+  <xacro:arg name="ee"            default="false"/>
   <xacro:arg name="ee_parent"     default="tool0"/>
-  <xacro:arg name="ee_z_offset"   default="+0.0"/>
-  <xacro:arg name="ee_rz"         default="+0.0"/>
-  <xacro:arg name="tcp_offset"    default="+0.05"/>
-  <!-- Include ur5e model -->
-  <xacro:include filename="$(find ur_description)/urdf/inc/ur5e_macro.xacro"/>
-  <xacro:ur5e_robot prefix="" />
+  <xacro:arg name="ee_z_offset"   default="+0.00"/>
+  <xacro:arg name="ee_rz"         default="+0.00"/>
+  <xacro:arg name="tcp_offset"    default="+0.00"/>
+  <!-- Include ur3e model -->
+  <xacro:include filename="$(find ur_description)/urdf/inc/ur3e_macro.xacro"/>
+  <xacro:ur3e_robot prefix="" />
   <!-- Fixed tcp gripper -->
   <link name="tcp_gripper"/>
   <joint name="tcp_gripper_joint" type="fixed">
     <origin xyz="0 0 $(arg tcp_offset)" rpy="0 0 0"/>
-    <parent link="$(arg ee_parent)"/>
+    <parent link="tool0"/>
     <child  link="tcp_gripper"/>
   </joint>
+  <!-- Add camera -->
+  <xacro:if value="$(arg camera)">
+    <!-- Fixed joint camera -->
+    <joint name="camera_robot_joint" type="fixed">
+      <origin xyz="$(arg cam_x_offset) $(arg cam_y_offset) $(arg cam_z_offset)"
+              rpy="$(arg cam_rx) $(arg cam_ry) $(arg cam_rz)"/>
+      <parent link="$(arg cam_parent)"/>
+      <child  link="camera_base_link"/>
+    </joint>
+    <!-- Import d435 xacro file -->
+    <xacro:include filename="$(find realsense2_description)/urdf/_d435.urdf.xacro" />
+    <link name="camera_base_link">
+      <collision>
+        <origin xyz="-0.0061 0.0 +0.0125" rpy="0 0 0"/>
+        <geometry>
+          <box size="0.0083 0.09 0.025"/>
+        </geometry>
+      </collision>
+    </link>
+    <xacro:sensor_d435 parent="camera_base_link" use_nominal_extrinsics="false" add_plug="false" use_mesh="true">
+      <origin xyz="0 0 0" rpy="0 0 0"/>
+    </xacro:sensor_d435>
+  </xacro:if>
+  <!-- Add end-effector -->
+  <xacro:if value="$(arg ee)">
+    <!-- Import Robotiq85Gripper -->
+    <xacro:include filename="$(find gripper)/models/robotiq_85.urdf.xacro"/>
+    <!-- Fixed joint gripper -->
+    <joint name="gripper_robot_joint" type="fixed">
+      <origin xyz="0 0 $(arg ee_z_offset)" rpy="0 0 $(arg ee_rz)"/>
+      <parent link="$(arg ee_parent)"/>
+      <child  link="robotiq_85_base_link"/>
+    </joint>
+  </xacro:if>
 </robot>

File: models/urdf/ur5.xacro (robot description, xacro)
@@ -1,8 +1,8 @@
 <?xml version="1.0"?>
-<robot xmlns:xacro="http://wiki.ros.org/xacro" name="ur5e_robot">
+<robot xmlns:xacro="http://wiki.ros.org/xacro" name="ur5_robot">
   <!--
-    This is a convenience top-level xacro which loads the macro for the UR10e
+    This is a convenience top-level xacro which loads the macro for the UR5
     which defines the default values for the various "parameters files"
-    parameters for a UR5e.
+    parameters for a UR5.
     This file is only useful when loading a stand-alone, completely isolated
     robot with only default values for all parameters such as the kinematics,
@@ -10,5 +10,5 @@
     This file is not intended to be integrated into a larger scene or other
     composite xacro.
-    Instead, xacro:include 'inc/ur5e_macro.xacro' and override the defaults
+    Instead, xacro:include 'inc/ur5_macro.xacro' and override the defaults
     for the arguments to that macro.
     Refer to 'inc/ur_macro.xacro' for more information.
@@ -16,25 +16,61 @@
   <!-- Args for starting ee tool position -->
     <!-- Args for starting camera position -->
+  <xacro:arg name="camera"        default="false"/>
   <xacro:arg name="cam_parent"    default="tool0"/>
-  <xacro:arg name="cam_x_offset"  default="+0.0"/>
-  <xacro:arg name="cam_y_offset"  default="+0.05"/>
-  <xacro:arg name="cam_z_offset"  default="+0.05"/>
-  <xacro:arg name="cam_rx"        default="+0.0"/>
+  <xacro:arg name="cam_x_offset"  default="+0.00"/>
+  <xacro:arg name="cam_y_offset"  default="+0.00"/>
+  <xacro:arg name="cam_z_offset"  default="+0.00"/>
+  <xacro:arg name="cam_rx"        default="+0.00"/>
   <xacro:arg name="cam_ry"        default="-1.570796327"/>
   <xacro:arg name="cam_rz"        default="-1.570796327"/>
   <!-- Args for starting gripper position -->
+  <xacro:arg name="ee"            default="false"/>
   <xacro:arg name="ee_parent"     default="tool0"/>
-  <xacro:arg name="ee_z_offset"   default="+0.0"/>
-  <xacro:arg name="ee_rz"         default="+0.0"/>
-  <xacro:arg name="tcp_offset"    default="+0.05"/>
-  <!-- Include ur5e model -->
-  <xacro:include filename="$(find ur_description)/urdf/inc/ur5e_macro.xacro"/>
-  <xacro:ur5e_robot prefix="" />
+  <xacro:arg name="ee_z_offset"   default="+0.00"/>
+  <xacro:arg name="ee_rz"         default="+0.00"/>
+  <xacro:arg name="tcp_offset"    default="+0.00"/>
+  <!-- Include ur5 model -->
+  <xacro:include filename="$(find ur_description)/urdf/inc/ur5_macro.xacro"/>
+  <xacro:ur5_robot prefix="" />
   <!-- Fixed tcp gripper -->
   <link name="tcp_gripper"/>
   <joint name="tcp_gripper_joint" type="fixed">
     <origin xyz="0 0 $(arg tcp_offset)" rpy="0 0 0"/>
-    <parent link="$(arg ee_parent)"/>
+    <parent link="tool0"/>
     <child  link="tcp_gripper"/>
   </joint>
+  <!-- Add camera -->
+  <xacro:if value="$(arg camera)">
+    <!-- Fixed joint camera -->
+    <joint name="camera_robot_joint" type="fixed">
+      <origin xyz="$(arg cam_x_offset) $(arg cam_y_offset) $(arg cam_z_offset)"
+              rpy="$(arg cam_rx) $(arg cam_ry) $(arg cam_rz)"/>
+      <parent link="$(arg cam_parent)"/>
+      <child  link="camera_base_link"/>
+    </joint>
+    <!-- Import d435 xacro file -->
+    <xacro:include filename="$(find realsense2_description)/urdf/_d435.urdf.xacro" />
+    <link name="camera_base_link">
+      <collision>
+        <origin xyz="-0.0061 0.0 +0.0125" rpy="0 0 0"/>
+        <geometry>
+          <box size="0.0083 0.09 0.025"/>
+        </geometry>
+      </collision>
+    </link>
+    <xacro:sensor_d435 parent="camera_base_link" use_nominal_extrinsics="false" add_plug="false" use_mesh="true">
+      <origin xyz="0 0 0" rpy="0 0 0"/>
+    </xacro:sensor_d435>
+  </xacro:if>
+  <!-- Add end-effector -->
+  <xacro:if value="$(arg ee)">
+    <!-- Import Robotiq85Gripper -->
+    <xacro:include filename="$(find gripper)/models/robotiq_85.urdf.xacro"/>
+    <!-- Fixed joint gripper -->
+    <joint name="gripper_robot_joint" type="fixed">
+      <origin xyz="0 0 $(arg ee_z_offset)" rpy="0 0 $(arg ee_rz)"/>
+      <parent link="$(arg ee_parent)"/>
+      <child  link="robotiq_85_base_link"/>
+    </joint>
+  </xacro:if>
 </robot>

File: models/urdf/ur5e.xacro (robot description, xacro)
@@ -2,5 +2,5 @@
 <robot xmlns:xacro="http://wiki.ros.org/xacro" name="ur5e_robot">
   <!--
-    This is a convenience top-level xacro which loads the macro for the UR10e
+    This is a convenience top-level xacro which loads the macro for the UR5e
     which defines the default values for the various "parameters files"
     parameters for a UR5e.
@@ -16,16 +16,18 @@
   <!-- Args for starting ee tool position -->
     <!-- Args for starting camera position -->
+  <xacro:arg name="camera"        default="false"/>
   <xacro:arg name="cam_parent"    default="tool0"/>
-  <xacro:arg name="cam_x_offset"  default="+0.0"/>
-  <xacro:arg name="cam_y_offset"  default="+0.05"/>
-  <xacro:arg name="cam_z_offset"  default="+0.05"/>
-  <xacro:arg name="cam_rx"        default="+0.0"/>
+  <xacro:arg name="cam_x_offset"  default="+0.00"/>
+  <xacro:arg name="cam_y_offset"  default="+0.00"/>
+  <xacro:arg name="cam_z_offset"  default="+0.00"/>
+  <xacro:arg name="cam_rx"        default="+0.00"/>
   <xacro:arg name="cam_ry"        default="-1.570796327"/>
   <xacro:arg name="cam_rz"        default="-1.570796327"/>
   <!-- Args for starting gripper position -->
+  <xacro:arg name="ee"            default="false"/>
   <xacro:arg name="ee_parent"     default="tool0"/>
-  <xacro:arg name="ee_z_offset"   default="+0.0"/>
-  <xacro:arg name="ee_rz"         default="+0.0"/>
-  <xacro:arg name="tcp_offset"    default="+0.05"/>
+  <xacro:arg name="ee_z_offset"   default="+0.00"/>
+  <xacro:arg name="ee_rz"         default="+0.00"/>
+  <xacro:arg name="tcp_offset"    default="+0.00"/>
   <!-- Include ur5e model -->
   <xacro:include filename="$(find ur_description)/urdf/inc/ur5e_macro.xacro"/>
@@ -35,6 +37,40 @@
   <joint name="tcp_gripper_joint" type="fixed">
     <origin xyz="0 0 $(arg tcp_offset)" rpy="0 0 0"/>
-    <parent link="$(arg ee_parent)"/>
+    <parent link="tool0"/>
     <child  link="tcp_gripper"/>
   </joint>
+  <!-- Add camera -->
+  <xacro:if value="$(arg camera)">
+    <!-- Fixed joint camera -->
+    <joint name="camera_robot_joint" type="fixed">
+      <origin xyz="$(arg cam_x_offset) $(arg cam_y_offset) $(arg cam_z_offset)"
+              rpy="$(arg cam_rx) $(arg cam_ry) $(arg cam_rz)"/>
+      <parent link="$(arg cam_parent)"/>
+      <child  link="camera_base_link"/>
+    </joint>
+    <!-- Import d435 xacro file -->
+    <xacro:include filename="$(find realsense2_description)/urdf/_d435.urdf.xacro" />
+    <link name="camera_base_link">
+      <collision>
+        <origin xyz="-0.0061 0.0 +0.0125" rpy="0 0 0"/>
+        <geometry>
+          <box size="0.0083 0.09 0.025"/>
+        </geometry>
+      </collision>
+    </link>
+    <xacro:sensor_d435 parent="camera_base_link" use_nominal_extrinsics="false" add_plug="false" use_mesh="true">
+      <origin xyz="0 0 0" rpy="0 0 0"/>
+    </xacro:sensor_d435>
+  </xacro:if>
+  <!-- Add end-effector -->
+  <xacro:if value="$(arg ee)">
+    <!-- Import Robotiq85Gripper -->
+    <xacro:include filename="$(find gripper)/models/robotiq_85.urdf.xacro"/>
+    <!-- Fixed joint gripper -->
+    <joint name="gripper_robot_joint" type="fixed">
+      <origin xyz="0 0 $(arg ee_z_offset)" rpy="0 0 $(arg ee_rz)"/>
+      <parent link="$(arg ee_parent)"/>
+      <child  link="robotiq_85_base_link"/>
+    </joint>
+  </xacro:if>
 </robot>
