Commit message: Added camera

File: models/urdf/ur_robotiq_85_gripper.urdf.xacro (robot description, xacro)
@@ -1,5 +1,5 @@
 <?xml version="1.0"?>
 <robot name="$(arg name)" xmlns:xacro="http://ros.org/wiki/xacro">
-  <xacro:include filename="$(find manipulators)/models/urdf/ur_robotiq_85_gripper_macro.xacro"/>
+    <xacro:include filename="$(find manipulators)/models/urdf/ur_robotiq_85_gripper_macro.xacro"/>
     <xacro:arg name="name" default="ur"/>
     <xacro:arg name="ur_type" default="ur5e"/>
@@ -7,4 +7,5 @@
     <xacro:arg name="joint_limits_parameters_file" default="$(find ur_description)/config/$(arg ur_type)/joint_limits.yaml"/>
     <xacro:arg name="kinematics_parameters_file" default="$(find ur_description)/config/$(arg ur_type)/default_kinematics.yaml"/>
+    <xacro:arg name="camera" default="true" />
     <link name="world" />
     <!--This will create the scene where the robot is located in-->
@@ -17,3 +18,16 @@
     >
     </xacro:ur_robotiq_85_gripper>
+    <xacro:property name="camera" value="$(arg camera)"/>
+    <xacro:if value="${camera}">
+        <xacro:include filename="$(find realsense2_description)/urdf/_d435i.urdf.xacro"/>
+        <link name="d435i_base_link" />
+        <joint name="tool0-d4351_base_link" type="fixed">
+            <parent link="tool0"/>
+            <child link="d435i_base_link"/>
+            <origin xyz="0 -0.09 0" rpy="0 -1.57 1.57"/>
+        </joint>
+        <xacro:sensor_d435i parent="d435i_base_link" name="camera">
+            <origin xyz="0 0 0" rpy="0 0 0" />
+        </xacro:sensor_d435i>
+    </xacro:if>
 </robot>

Commit message: joint goal in joystick control

File: models/urdf/ur_robotiq_85_gripper.urdf.xacro (robot description, xacro)
@@ -25,5 +25,5 @@
             <parent link="tool0"/>
             <child link="d435i_base_link"/>
-            <origin xyz="0 -0.09 0" rpy="0 -1.57 1.57"/>
+            <origin xyz="0 -0.0775 0.024" rpy="0 -1.57 1.57"/>
         </joint>
         <xacro:sensor_d435i parent="d435i_base_link" name="camera">

Commit message: More real control implementations

File: models/urdf/ur_robotiq_85_gripper.urdf.xacro (robot description, xacro)
@@ -31,3 +31,23 @@
         </xacro:sensor_d435i>
     </xacro:if>
+    <link name="floor">
+        <visual>
+            <geometry>
+                <box size="10 10 0.01"/>
+            </geometry>
+            <material name="">
+                <color rgba="0.8 0.1 0.1 0.4"/>
+            </material>
+        </visual>
+        <collision>
+            <geometry>
+                <box size="10 10 0.01"/>
+            </geometry>
+        </collision>
+    </link>
+    <joint name="world_floor" type="fixed">
+        <parent link="world"/>
+        <child link="floor"/>
+        <origin xyz="0 0 -0.005" rpy="0 0 0"/>
+    </joint>
 </robot>
