Commit message: Fixed bug in eecam urdf files which prevented gripper argument to be set to false

File: models/urdf/ur10e_robotiq_85_gripper.urdf.xacro (robot description, xacro)
@@ -1,4 +1,6 @@
 <?xml version="1.0"?>
 <robot name="$(arg name)" xmlns:xacro="http://ros.org/wiki/xacro">
+    <!-- Robot URDF file-->
+    <xacro:include filename="$(find ur_description)/urdf/ur_macro.xacro"/>
     <!-- Robot Arguments -->
     <xacro:arg name="name" default="ur"/>
@@ -14,4 +16,17 @@
     <xacro:property name="gripper"  value="$(arg gripper)"/>
     <xacro:property name="gfloor"   value="$(arg gfloor)"/>
+    <!-- Create the manipulator -->
+    <link name="world"/>
+    <xacro:ur_robot
+        parent="world"
+        name="$(arg name)"
+        tf_prefix="$(arg tf_prefix)"
+        joint_limits_parameters_file="$(arg joint_limits_parameters_file)"
+        kinematics_parameters_file="$(arg kinematics_parameters_file)"
+        physical_parameters_file="$(find ur_description)/config/$(arg ur_type)/physical_parameters.yaml"
+        visual_parameters_file="$(find ur_description)/config/$(arg ur_type)/visual_parameters.yaml"
+    >
+        <origin xyz="0 0 0" rpy="0 0 0" />
+    </xacro:ur_robot>
     <!-- Gripper inclusion -->
     <xacro:if value="${gripper}">
@@ -19,8 +34,4 @@
         <xacro:ur_robotiq_85_gripper
             tf_prefix="$(arg tf_prefix)"
-            robot_name="$(arg name)"
-            ur_type="$(arg ur_type)"
-            joint_limits_parameters_file="$(arg joint_limits_parameters_file)"
-            kinematics_parameters_file="$(arg kinematics_parameters_file)"
         />
     </xacro:if>

File: models/urdf/ur5e_robotiq_85_gripper.urdf.xacro (robot description, xacro)
@@ -1,4 +1,6 @@
 <?xml version="1.0"?>
 <robot name="$(arg name)" xmlns:xacro="http://ros.org/wiki/xacro">
+    <!-- Robot URDF file-->
+    <xacro:include filename="$(find ur_description)/urdf/ur_macro.xacro"/>
     <!-- Robot Arguments -->
     <xacro:arg name="name" default="ur"/>
@@ -14,4 +16,17 @@
     <xacro:property name="gripper"  value="$(arg gripper)"/>
     <xacro:property name="gfloor"   value="$(arg gfloor)"/>
+    <!-- Create the manipulator -->
+    <link name="world"/>
+    <xacro:ur_robot
+        parent="world"
+        name="$(arg name)"
+        tf_prefix="$(arg tf_prefix)"
+        joint_limits_parameters_file="$(arg joint_limits_parameters_file)"
+        kinematics_parameters_file="$(arg kinematics_parameters_file)"
+        physical_parameters_file="$(find ur_description)/config/$(arg ur_type)/physical_parameters.yaml"
+        visual_parameters_file="$(find ur_description)/config/$(arg ur_type)/visual_parameters.yaml"
+    >
+        <origin xyz="0 0 0" rpy="0 0 0" />
+    </xacro:ur_robot>
     <!-- Gripper inclusion -->
     <xacro:if value="${gripper}">
@@ -19,8 +34,4 @@
         <xacro:ur_robotiq_85_gripper
             tf_prefix="$(arg tf_prefix)"
-            robot_name="$(arg name)"
-            ur_type="$(arg ur_type)"
-            joint_limits_parameters_file="$(arg joint_limits_parameters_file)"
-            kinematics_parameters_file="$(arg kinematics_parameters_file)"
         />
     </xacro:if>

File: models/urdf/ur_robotiq_85_gripper_macro.xacro (robot description, xacro)
@@ -1,17 +1,8 @@
 <?xml version="1.0"?>
 <robot xmlns:xacro="http://ros.org/wiki/xacro">
-    <!-- Robot URDF file-->
-    <xacro:include filename="$(find ur_description)/urdf/ur_macro.xacro"/>
     <!-- Robotiq 85 Gripper URDF file -->
     <xacro:include filename="$(find robotiq_85_description)/urdf/robotiq_85_gripper_macro.urdf.xacro"/>
     <!-- Gripper macro definition -->
-    <xacro:macro name="ur_robotiq_85_gripper" params="
-        robot_name
-        tf_prefix
-        ur_type
-        joint_limits_parameters_file
-        kinematics_parameters_file
-        "
-    >
+    <xacro:macro name="ur_robotiq_85_gripper" params="tf_prefix">
         <!-- Create a link for the 'tool0' as parent for the gripper -->
         <xacro:robotiq_85_gripper
@@ -30,17 +21,4 @@
             <child link="tcp_gripper" />
         </joint>
-        <!--This will create the specific robot-->
-        <link name="world"/>
-        <xacro:ur_robot
-            parent="world"
-            name="${robot_name}"
-            tf_prefix="${tf_prefix}"
-            joint_limits_parameters_file="${joint_limits_parameters_file}"
-            kinematics_parameters_file="${kinematics_parameters_file}"
-            physical_parameters_file="$(find ur_description)/config/${ur_type}/physical_parameters.yaml"
-            visual_parameters_file="$(find ur_description)/config/${ur_type}/visual_parameters.yaml"
-        >
-            <origin xyz="0 0 0" rpy="0 0 0" />
-        </xacro:ur_robot>
   </xacro:macro>
 </robot>

Commit message: Merge

File: models/urdf/ur10e_robotiq_85_gripper.urdf.xacro (robot description, xacro)
@@ -17,7 +17,7 @@
     <xacro:property name="gfloor"   value="$(arg gfloor)"/>
     <!-- Create the manipulator -->
-    <link name="world"/>
+    <link name="world_ur"/>
     <xacro:ur_robot
-        parent="world"
+        parent="world_ur"
         name="$(arg name)"
         tf_prefix="$(arg tf_prefix)"
