Commit message: modifiche

File: models/urdf/ur5e_robotiq_85_gripper.urdf.xacro (robot description, xacro)
@@ -100,5 +100,5 @@
             <parent link="tool0"/>
             <child link="tcp_gripper"/>
-            <origin xyz="0 0 0.145" rpy="0 0 0"/>
+            <origin xyz="0 0 0.145" rpy="0 0 0.21"/>
         </joint>
     </xacro:if>

Commit message: Fixed typos over ur5e_eecam planner config

File: models/urdf/ur5e_robotiq_85_gripper.urdf.xacro (robot description, xacro)
@@ -10,16 +10,18 @@
     <xacro:arg name="kinematics_parameters_file" default="$(find ur_description)/config/$(arg ur_type)/default_kinematics.yaml"/>
     <!-- Additional objects Arguments -->
-    <xacro:arg name="camera"                   default="true"/>
-    <xacro:arg name="gripper"                  default="true"/>
-    <xacro:arg name="gfloor"                   default="false"/>
-    <xacro:arg name="gripper_collision_box"    default="false"/>
-    <xacro:property name="camera"                value="$(arg camera)"/>
-    <xacro:property name="gripper"               value="$(arg gripper)"/>
-    <xacro:property name="gfloor"                value="$(arg gfloor)"/>
-    <xacro:property name="gripper_collision_box" value="$(arg gripper_collision_box)"/>
+    <xacro:arg name="camera"                        default="true"/>
+    <xacro:arg name="gripper"                       default="true"/>
+    <xacro:arg name="gfloor"                        default="false"/>
+    <xacro:arg name="gripper_collision_box"         default="false"/>
+    <xacro:arg name="tcp_offset"                    default="0.148"/>
+    <xacro:arg name="tcp_z_rot"                     default="0.0"/>
+    <xacro:property name="camera"                   value="$(arg camera)"/>
+    <xacro:property name="gripper"                  value="$(arg gripper)"/>
+    <xacro:property name="gfloor"                   value="$(arg gfloor)"/>
+    <xacro:property name="gripper_collision_box"    value="$(arg gripper_collision_box)"/>
     <!-- Create the manipulator -->
-    <link name="world"/>
+    <link name="world_ur"/>
     <xacro:ur_robot
-        parent="world"
+        parent="world_ur"
         name="$(arg name)"
         tf_prefix="$(arg tf_prefix)"
@@ -42,5 +44,5 @@
         <xacro:include filename="$(find realsense2_description)/urdf/_d435i.urdf.xacro"/>
         <link name="d435i_base_link" />
-        <joint name="tool0-d4351_base_link" type="fixed">
+        <joint name="tool0-d435i_base_link" type="fixed">
             <parent link="tool0"/>
             <child link="d435i_base_link"/>
@@ -69,5 +71,5 @@
         </link>
         <joint name="world_floor" type="fixed">
-            <parent link="world"/>
+            <parent link="world_ur"/>
             <child link="floor"/>
             <origin xyz="0 0 -0.005" rpy="0 0 0"/>
@@ -94,5 +96,5 @@
             <parent link="tool0"/>
             <child link="ee_collision_box"/>
-            <origin xyz="0 -0.04 0.080" rpy="0 0 0"/>
+            <origin xyz="0 0.0 0.080" rpy="0 0 0"/>
         </joint>
         <link name="tcp_gripper" />
@@ -100,5 +102,5 @@
             <parent link="tool0"/>
             <child link="tcp_gripper"/>
-            <origin xyz="0 0 0.145" rpy="0 0 0.21"/>
+            <origin xyz="0 0 $(arg tcp_offset)" rpy="0 0 $(arg tcp_z_rot)"/>
         </joint>
     </xacro:if>

Commit message: Solved manipulator urdf for ur5e

File: models/urdf/ur5e_robotiq_85_gripper.urdf.xacro (robot description, xacro)
@@ -20,4 +20,6 @@
     <xacro:property name="gfloor"                   value="$(arg gfloor)"/>
     <xacro:property name="gripper_collision_box"    value="$(arg gripper_collision_box)"/>
+    <xacro:property name="tcp_offset"               value="$(arg tcp_offset)"/>
+    <xacro:property name="tcp_z_rot"                value="$(arg tcp_z_rot)"/>
     <!-- Create the manipulator -->
     <link name="world_ur"/>
@@ -47,5 +49,6 @@
             <parent link="tool0"/>
             <child link="d435i_base_link"/>
-            <origin xyz="0 -0.0775 0.024" rpy="0 -1.57 1.57"/>
+            <!-- <origin xyz="0 -0.0775 0.024" rpy="0 -1.57 1.57"/> -->
+            <origin xyz="0.08 0 -0.04" rpy="0 -1.57 3.14"/>
         </joint>
         <xacro:sensor_d435i parent="d435i_base_link" name="ee_cam">
@@ -56,5 +59,6 @@
     <xacro:if value="${gfloor}">
         <link name="floor">
-            <visual>
+            <visual> <!-- floor -->
+                <origin xyz="0.0 0.0 -0.40" rpy="0 0 0"/>
                 <geometry>
                     <box size="10 10 0.01"/>
@@ -64,4 +68,5 @@
                 </material>
             </visual>
+            <origin xyz="0.0 0.0 -0.40" rpy="0 0 0"/>
             <collision>
                 <geometry>
@@ -69,9 +74,40 @@
                 </geometry>
             </collision>
+            <visual>
+                <geometry>
+                    <box size="1.0 0.7 0.5"/> <!-- box sotto -->
+                </geometry>
+                <origin xyz="-0.25 0.0 -0.25" rpy="0 0 0"/>
+                <material name="">
+                        <color rgba="1.0 1.0 1.0 1.0"/>
+                </material>
+            </visual>
+            <visual>
+                <geometry>
+                    <box size="0.6 0.7 0.4"/> <!-- box sopra -->
+                </geometry>
+                <origin xyz="-0.4 0.0 0.2" rpy="0 0 0"/>
+                <material name="">
+                    <color rgba="1.0 1.0 1.0 1.0"/>
+                </material>
+            </visual>
+            <collision>
+                <geometry>
+                    <box size="1.0 0.7 0.5"/> <!-- box sotto -->
+                </geometry>
+                <origin xyz="-0.25 0.0 -0.25" rpy="0 0 0"/>
+            </collision>
+            <collision>
+                <geometry>
+                    <box size="0.6 0.7 0.4"/> <!-- box sopra -->
+                </geometry>
+                <origin xyz="-0.4 0.0 0.2" rpy="0 0 0"/>
+            </collision>
         </link>
         <joint name="world_floor" type="fixed">
-            <parent link="world_ur"/>
+            <parent link="base_link"/>
             <child link="floor"/>
-            <origin xyz="0 0 -0.005" rpy="0 0 0"/>
+            <!-- <origin xyz="0 0 -0.005" rpy="0 0 0"/> -->
+            <origin xyz="0 0 0" rpy="0 0 0"/>
         </joint>
     </xacro:if>
@@ -80,6 +116,7 @@
         <link name="ee_collision_box">
             <visual>
+                <origin xyz="0 0 0" rpy="0 0 0"/>
                 <geometry>
-                    <box size="0.130 0.170 0.160"/>
+                    <box size="0.130 0.170 $(arg tcp_offset)"/>  <!-- 0.130 0.170 0.160 or 0.270 0.180 $(arg tcp_offset)-->
                 </geometry>
                 <material name="">
@@ -88,6 +125,7 @@
             </visual>
             <collision>
+                <origin xyz="0 0 0" rpy="0 0 0"/>
                 <geometry>
-                    <box size="0.130 0.170 0.160"/>
+                    <box size="0.130 0.170 $(arg tcp_offset)"/>  <!-- 0.130 0.170 0.160 or 0.270 0.180 $(arg tcp_offset) -->
                 </geometry>
             </collision>
@@ -96,5 +134,5 @@
             <parent link="tool0"/>
             <child link="ee_collision_box"/>
-            <origin xyz="0 0.0 0.080" rpy="0 0 0"/>
+            <origin xyz="0 0.0 0.080 " rpy="0 0 0"/> <!-- 0 0.0 0.080  0.05 0.0 0.040 -->
         </joint>
         <link name="tcp_gripper" />

Commit message: Solved body collision bug

File: models/urdf/ur5e_robotiq_85_gripper.urdf.xacro (robot description, xacro)
@@ -68,6 +68,6 @@
                 </material>
             </visual>
-            <origin xyz="0.0 0.0 -0.40" rpy="0 0 0"/>
             <collision>
+                <origin xyz="0.0 0.0 -0.40" rpy="0 0 0"/>
                 <geometry>
                     <box size="10 10 0.01"/>
