Commit message: Dynamic planner functions restored (collision boxes, constraints, etc.), launch file improvements

File: models/urdf/ur5e_mobile.urdf.xacro (robot description, xacro)
@@ -12,5 +12,5 @@
     <xacro:arg name="camera"                        default="true"/>
     <xacro:arg name="gripper"                       default="true"/>
-    <xacro:arg name="gfloor"                        default="false"/>
+    <xacro:arg name="gfloor"                        default="true"/>
     <xacro:arg name="gripper_collision_box"         default="false"/>
     <xacro:arg name="tcp_offset"                    default="0.148"/>
@@ -20,4 +20,6 @@
     <xacro:property name="gfloor"                   value="$(arg gfloor)"/>
     <xacro:property name="gripper_collision_box"    value="$(arg gripper_collision_box)"/>
+    <xacro:property name="tcp_offset"               value="$(arg tcp_offset)"/>
+    <xacro:property name="tcp_z_rot"                value="$(arg tcp_z_rot)"/>
     <!-- Create the manipulator -->
     <link name="world_ur"/>
@@ -47,5 +49,6 @@
             <parent link="tool0"/>
             <child link="d435i_base_link"/>
-            <origin xyz="0 -0.0775 0.024" rpy="0 -1.57 1.57"/>
+            <!-- <origin xyz="0 -0.0775 0.024" rpy="0 -1.57 1.57"/> -->
+            <origin xyz="0.08 0 -0.04" rpy="0 -1.57 3.14"/>
         </joint>
         <xacro:sensor_d435i parent="d435i_base_link" name="ee_cam">
@@ -56,5 +59,6 @@
     <xacro:if value="${gfloor}">
         <link name="floor">
-            <visual>
+            <visual> <!-- floor -->
+                <origin xyz="0.0 0.0 -0.40" rpy="0 0 0"/>
                 <geometry>
                     <box size="10 10 0.01"/>
@@ -65,13 +69,45 @@
             </visual>
             <collision>
+                <origin xyz="0.0 0.0 -0.40" rpy="0 0 0"/>
                 <geometry>
                     <box size="10 10 0.01"/>
                 </geometry>
             </collision>
+            <visual>
+                <geometry>
+                    <box size="1.0 0.7 0.5"/> <!-- box sotto -->
+                </geometry>
+                <origin xyz="-0.25 0.0 -0.25" rpy="0 0 0"/>
+                <material name="">
+                        <color rgba="1.0 1.0 1.0 1.0"/>
+                </material>
+            </visual>
+            <visual>
+                <geometry>
+                    <box size="0.6 0.7 0.4"/> <!-- box sopra -->
+                </geometry>
+                <origin xyz="-0.4 0.0 0.2" rpy="0 0 0"/>
+                <material name="">
+                    <color rgba="1.0 1.0 1.0 1.0"/>
+                </material>
+            </visual>
+            <collision>
+                <geometry>
+                    <box size="1.0 0.7 0.5"/> <!-- box sotto -->
+                </geometry>
+                <origin xyz="-0.25 0.0 -0.25" rpy="0 0 0"/>
+            </collision>
+            <collision>
+                <geometry>
+                    <box size="0.6 0.7 0.4"/> <!-- box sopra -->
+                </geometry>
+                <origin xyz="-0.4 0.0 0.2" rpy="0 0 0"/>
+            </collision>
         </link>
         <joint name="world_floor" type="fixed">
-            <parent link="world_ur"/>
+            <parent link="base_link"/>
             <child link="floor"/>
-            <origin xyz="0 0 -0.005" rpy="0 0 0"/>
+            <!-- <origin xyz="0 0 -0.005" rpy="0 0 0"/> -->
+            <origin xyz="0 0 0" rpy="0 0 0"/>
         </joint>
     </xacro:if>
@@ -80,6 +116,7 @@
         <link name="ee_collision_box">
             <visual>
+                <origin xyz="0 0 0" rpy="0 0 0"/>
                 <geometry>
-                    <box size="0.130 0.170 0.160"/>
+                    <box size="0.130 0.170 $(arg tcp_offset)"/>  <!-- 0.130 0.170 0.160 or 0.270 0.180 $(arg tcp_offset)-->
                 </geometry>
                 <material name="">
@@ -88,6 +125,7 @@
             </visual>
             <collision>
+                <origin xyz="0 0 0" rpy="0 0 0"/>
                 <geometry>
-                    <box size="0.130 0.170 0.160"/>
+                    <box size="0.130 0.170 $(arg tcp_offset)"/>  <!-- 0.130 0.170 0.160 or 0.270 0.180 $(arg tcp_offset) -->
                 </geometry>
             </collision>
@@ -96,5 +134,5 @@
             <parent link="tool0"/>
             <child link="ee_collision_box"/>
-            <origin xyz="0 0.0 0.080" rpy="0 0 0"/>
+            <origin xyz="0 0.0 0.080 " rpy="0 0 0"/> <!-- 0 0.0 0.080  0.05 0.0 0.040 -->
         </joint>
         <link name="tcp_gripper" />
