Commit message: Merged ros2-humble lastest changes

File: models/urdf/ur5e_eecam.urdf.xacro (robot description, xacro)
@@ -13,6 +13,6 @@
     <xacro:arg name="gfloor"                        default="true"/>
     <xacro:arg name="gripper_collision_box"         default="true"/>
-    <xacro:arg name="tcp_offset"                    default="0.148"/>
-    <xacro:arg name="tcp_z_rot"                     default="0.3"/>
+    <xacro:arg name="tcp_offset"                    default="0.160"/>
+    <xacro:arg name="tcp_z_rot"                     default="0.300"/>
     <xacro:property name="camera"                   value="$(arg camera)"/>
     <xacro:property name="gripper"                  value="$(arg gripper)"/>
@@ -48,6 +48,5 @@
             <parent link="tool0"/>
             <child link="d435i_base_link"/>
-            <!-- <origin xyz="0 -0.0775 0.024" rpy="0 -1.57 1.57"/> -->
-            <origin xyz="0.08 0 -0.04" rpy="0 -1.57 3.14"/>
+            <origin xyz="0 -0.0775 0.024" rpy="0 -1.57 1.57"/>
         </joint>
         <xacro:sensor_d435i parent="d435i_base_link" name="ee_cam">
@@ -73,40 +72,9 @@
                 </geometry>
             </collision>
-            <visual>
-                <geometry>
-                    <box size="1.0 0.7 0.5"/> <!-- box sotto -->
-                </geometry>
-                <origin xyz="-0.25 0.0 -0.25" rpy="0 0 0"/>
-                <material name="">
-                        <color rgba="1.0 1.0 1.0 1.0"/>
-                </material>
-            </visual>
-            <visual>
-                <geometry>
-                    <box size="0.6 0.7 0.4"/> <!-- box sopra -->
-                </geometry>
-                <origin xyz="-0.4 0.0 0.2" rpy="0 0 0"/>
-                <material name="">
-                    <color rgba="1.0 1.0 1.0 1.0"/>
-                </material>
-            </visual>
-            <collision>
-                <geometry>
-                    <box size="1.0 0.7 0.5"/> <!-- box sotto -->
-                </geometry>
-                <origin xyz="-0.25 0.0 -0.25" rpy="0 0 0"/>
-            </collision>
-            <collision>
-                <geometry>
-                    <box size="0.6 0.7 0.4"/> <!-- box sopra -->
-                </geometry>
-                <origin xyz="-0.4 0.0 0.2" rpy="0 0 0"/>
-            </collision>
         </link>
         <joint name="world_floor" type="fixed">
             <parent link="base_link"/>
             <child link="floor"/>
-            <!-- <origin xyz="0 0 -0.005" rpy="0 0 0"/> -->
-            <origin xyz="0 0 0" rpy="0 0 0"/>
+            <origin xyz="0 0 -0.005" rpy="0 0 0"/>
         </joint>
     </xacro:if>
@@ -117,5 +85,5 @@
                 <origin xyz="0 0 0" rpy="0 0 0"/>
                 <geometry>
-                    <box size="0.130 0.170 $(arg tcp_offset)"/>  <!-- 0.130 0.170 0.160 or 0.270 0.180 $(arg tcp_offset)-->
+                    <box size="0.130 0.170 $(arg tcp_offset)"/>
                 </geometry>
                 <material name="">
@@ -126,5 +94,5 @@
                 <origin xyz="0 0 0" rpy="0 0 0"/>
                 <geometry>
-                    <box size="0.130 0.170 $(arg tcp_offset)"/>  <!-- 0.130 0.170 0.160 or 0.270 0.180 $(arg tcp_offset) -->
+                    <box size="0.130 0.170 $(arg tcp_offset)"/>
                 </geometry>
             </collision>
@@ -133,5 +101,5 @@
             <parent link="tool0"/>
             <child link="ee_collision_box"/>
-            <origin xyz="0 0.0 0.080 " rpy="0 0 0"/> <!-- 0 0.0 0.080  0.05 0.0 0.040 -->
+            <origin xyz="0 0.0 0.080 " rpy="0 0 0"/>
         </joint>
         <link name="tcp_gripper" />

File: models/urdf/ur5e_mobile.urdf.xacro (robot description, xacro)
@@ -49,5 +49,4 @@
             <parent link="tool0"/>
             <child link="d435i_base_link"/>
-            <!-- <origin xyz="0 -0.0775 0.024" rpy="0 -1.57 1.57"/> -->
             <origin xyz="0.08 0 -0.04" rpy="0 -1.57 3.14"/>
         </joint>
@@ -108,5 +107,4 @@
             <parent link="base_link"/>
             <child link="floor"/>
-            <!-- <origin xyz="0 0 -0.005" rpy="0 0 0"/> -->
             <origin xyz="0 0 0" rpy="0 0 0"/>
         </joint>
@@ -118,5 +116,5 @@
                 <origin xyz="0 0 0" rpy="0 0 0"/>
                 <geometry>
-                    <box size="0.130 0.170 $(arg tcp_offset)"/>  <!-- 0.130 0.170 0.160 or 0.270 0.180 $(arg tcp_offset)-->
+                    <box size="0.130 0.170 $(arg tcp_offset)"/>
                 </geometry>
                 <material name="">
@@ -127,5 +125,5 @@
                 <origin xyz="0 0 0" rpy="0 0 0"/>
                 <geometry>
-                    <box size="0.130 0.170 $(arg tcp_offset)"/>  <!-- 0.130 0.170 0.160 or 0.270 0.180 $(arg tcp_offset) -->
+                    <box size="0.130 0.170 $(arg tcp_offset)"/>
                 </geometry>
             </collision>
@@ -134,5 +132,5 @@
             <parent link="tool0"/>
             <child link="ee_collision_box"/>
-            <origin xyz="0 0.0 0.080 " rpy="0 0 0"/> <!-- 0 0.0 0.080  0.05 0.0 0.040 -->
+            <origin xyz="0 0.0 0.080 " rpy="0 0 0"/>
         </joint>
         <link name="tcp_gripper" />
