Commit message: Updated driver with ZOH of joint state safe feedback. Added correct tracking of gripper, camera and tcp gripper on urdf of ur5e/ur10e mobile and ee cam. Updated manipulator limits on ur5e/ur10e mobile and ee cam.

File: models/urdf/ur10e_eecam.urdf.xacro (robot description, xacro)
@@ -10,10 +10,16 @@
     <xacro:arg name="kinematics_parameters_file" default="$(find ur_description)/config/$(arg ur_type)/default_kinematics.yaml"/>
     <!-- Additional objects Arguments -->
-    <xacro:arg name="camera"    default="true"/>
-    <xacro:arg name="gripper"   default="true"/>
-    <xacro:arg name="gfloor"    default="false"/>
-    <xacro:property name="camera"   value="$(arg camera)"/>
-    <xacro:property name="gripper"  value="$(arg gripper)"/>
-    <xacro:property name="gfloor"   value="$(arg gfloor)"/>
+    <xacro:arg name="camera"                        default="true"/>
+    <xacro:arg name="gripper"                       default="true"/>
+    <xacro:arg name="gfloor"                        default="true"/>
+    <xacro:arg name="gripper_collision_box"         default="false"/>
+    <xacro:arg name="tcp_offset"                    default="0.148"/>
+    <xacro:arg name="tcp_z_rot"                     default="0.0"/>
+    <xacro:property name="camera"                   value="$(arg camera)"/>
+    <xacro:property name="gripper"                  value="$(arg gripper)"/>
+    <xacro:property name="gfloor"                   value="$(arg gfloor)"/>
+    <xacro:property name="gripper_collision_box"    value="$(arg gripper_collision_box)"/>
+    <xacro:property name="tcp_offset"               value="$(arg tcp_offset)"/>
+    <xacro:property name="tcp_z_rot"                value="$(arg tcp_z_rot)"/>
     <!-- Create the manipulator -->
     <link name="world_ur"/>
@@ -39,12 +45,18 @@
     <xacro:if value="${camera}">
         <xacro:include filename="$(find realsense2_description)/urdf/_d435i.urdf.xacro"/>
+        <link name="camera_mount" />
+        <joint name="tcp_gripper-camera_mount" type="fixed">
+            <parent link="tcp_gripper"/>
+            <child link="camera_mount"/>
+            <origin xyz="-0.070 0 -0.135" rpy="0 $(arg camera_pitch) 0"/>
+        </joint>
         <link name="d435i_base_link" />
-        <joint name="tool0-d4351_base_link" type="fixed">
-            <parent link="tool0"/>
+        <joint name="camera_mount-d435i_base_link" type="fixed">
+            <parent link="camera_mount"/>
             <child link="d435i_base_link"/>
-            <origin xyz="0 -0.0775 0.024" rpy="0 -1.57 1.57"/>
+            <origin xyz="0 0 0.021" rpy="0 0 0"/>
         </joint>
         <xacro:sensor_d435i parent="d435i_base_link" name="ee_cam">
-            <origin xyz="0 0 0" rpy="0 0 0" />
+            <origin xyz="0 0 0" rpy="0 -1.57 0" />
         </xacro:sensor_d435i>
     </xacro:if>
@@ -72,3 +84,34 @@
         </joint>
     </xacro:if>
+    <!-- Gripper collision box -->
+    <xacro:if value="${gripper_collision_box}">
+        <link name="ee_collision_box">
+            <visual>
+                <origin xyz="0 0 0" rpy="0 0 0"/>
+                <geometry>
+                    <box size="0.130 0.170 $(arg tcp_offset)"/>
+                </geometry>
+                <material name="">
+                    <color rgba="0.8 0.1 0.1 0.4"/>
+                </material>
+            </visual>
+            <collision>
+                <origin xyz="0 0 0" rpy="0 0 0"/>
+                <geometry>
+                    <box size="0.130 0.170 $(arg tcp_offset)"/>
+                </geometry>
+            </collision>
+            <joint name="tool0-ee_collision_box" type="fixed">
+                <parent link="tool0"/>
+                <child link="ee_collision_box"/>
+                <origin xyz="0 0.0 0.080 " rpy="0 0 0"/>
+            </joint>
+        </link>
+    </xacro:if>
+    <link name="tcp_gripper" />
+    <joint name="tool0-tcp_gripper" type="fixed">
+        <parent link="tool0"/>
+        <child link="tcp_gripper"/>
+        <origin xyz="0 0 $(arg tcp_offset)" rpy="0 0 $(arg tcp_z_rot)"/>
+    </joint>
 </robot>

File: models/urdf/ur5e_eecam.urdf.xacro (robot description, xacro)
@@ -9,12 +9,14 @@
     <xacro:arg name="kinematics_parameters_file" default="$(find ur_description)/config/ur5e/default_kinematics.yaml"/>
     <!-- Additional objects Arguments -->
-    <xacro:arg name="camera"                        default="true"/>
+    <xacro:arg name="camera"                        default="false"/>
     <xacro:arg name="gripper"                       default="false"/>
-    <xacro:arg name="gfloor"                        default="true"/>
-    <xacro:arg name="gripper_collision_box"         default="true"/>
+    <xacro:arg name="gfloor"                        default="false"/>
+    <xacro:arg name="gripper_collision_box"         default="false"/>
     <xacro:arg name="back_wall"                     default="false"/>
-    <xacro:arg name="tcp_offset"                    default="0.160"/>
-    <xacro:arg name="tcp_z_rot"                     default="1.866"/>
+    <!-- <xacro:arg name="tcp_offset"                    default="0.148"/> -->
+    <xacro:arg name="tcp_offset"                    default="0.0"/>
+    <xacro:arg name="tcp_z_rot"                     default="0.0"/>
     <xacro:arg name="camera_pitch"                  default="0.41"/>
+    <!-- <xacro:arg name="tcp_z_rot"                     default="1.866"/> -->
     <xacro:property name="camera"                   value="$(arg camera)"/>
     <xacro:property name="gripper"                  value="$(arg gripper)"/>
@@ -44,4 +46,11 @@
         />
     </xacro:if>
+    <!-- TCP gripper inclusion -->
+    <link name="tcp_gripper" />
+    <joint name="tool0-tcp_gripper" type="fixed">
+        <parent link="tool0"/>
+        <child link="tcp_gripper"/>
+        <origin xyz="0 0 $(arg tcp_offset)" rpy="0 0 $(arg tcp_z_rot)"/>
+    </joint>
     <!-- Camera inclusion -->
     <xacro:if value="${camera}">
@@ -130,16 +139,16 @@
                 </geometry>
             </collision>
+            <joint name="tool0-ee_collision_box" type="fixed">
+                <parent link="tool0"/>
+                <child link="ee_collision_box"/>
+                <origin xyz="0 0.0 0.080 " rpy="0 0 0"/>
+            </joint>
         </link>
-        <joint name="tool0-ee_collision_box" type="fixed">
-            <parent link="tool0"/>
-            <child link="ee_collision_box"/>
-            <origin xyz="0 0.0 0.080 " rpy="0 0 0"/>
-        </joint>
-        <link name="tcp_gripper" />
-        <joint name="tool0-tcp_gripper" type="fixed">
-            <parent link="tool0"/>
-            <child link="tcp_gripper"/>
-            <origin xyz="0 0 $(arg tcp_offset)" rpy="0 0 $(arg tcp_z_rot)"/>
-        </joint>
     </xacro:if>
+    <link name="tcp_gripper" />
+    <joint name="tool0-ee_collision_box" type="fixed">
+        <parent link="tool0"/>
+        <child link="ee_collision_box"/>
+        <origin xyz="0 0.0 0.080 " rpy="0 0 0"/>
+    </joint>
 </robot>

File: models/urdf/ur5e_mobile.urdf.xacro (robot description, xacro)
@@ -45,12 +45,18 @@
     <xacro:if value="${camera}">
         <xacro:include filename="$(find realsense2_description)/urdf/_d435i.urdf.xacro"/>
+        <link name="camera_mount" />
+        <joint name="tcp_gripper-camera_mount" type="fixed">
+            <parent link="tcp_gripper"/>
+            <child link="camera_mount"/>
+            <origin xyz="-0.070 0 -0.135" rpy="0 $(arg camera_pitch) 0"/>
+        </joint>
         <link name="d435i_base_link" />
-        <joint name="tool0-d435i_base_link" type="fixed">
-            <parent link="tool0"/>
+        <joint name="camera_mount-d435i_base_link" type="fixed">
+            <parent link="camera_mount"/>
             <child link="d435i_base_link"/>
-            <origin xyz="0.08 0 -0.04" rpy="0 -1.57 3.14"/>
+            <origin xyz="0 0 0.021" rpy="0 0 0"/>
         </joint>
         <xacro:sensor_d435i parent="d435i_base_link" name="ee_cam">
-            <origin xyz="0 0 0" rpy="0 0 0" />
+            <origin xyz="0 0 0" rpy="0 -1.57 0" />
         </xacro:sensor_d435i>
     </xacro:if>
@@ -107,5 +113,5 @@
             <parent link="base_link"/>
             <child link="floor"/>
-            <origin xyz="0 0 0" rpy="0 0 0"/>
+            <origin xyz="0 0 -0.005" rpy="0 0 0"/>
         </joint>
     </xacro:if>
@@ -128,16 +134,16 @@
                 </geometry>
             </collision>
+            <joint name="tool0-ee_collision_box" type="fixed">
+                <parent link="tool0"/>
+                <child link="ee_collision_box"/>
+                <origin xyz="0 0.0 0.080 " rpy="0 0 0"/>
+            </joint>
         </link>
-        <joint name="tool0-ee_collision_box" type="fixed">
-            <parent link="tool0"/>
-            <child link="ee_collision_box"/>
-            <origin xyz="0 0.0 0.080 " rpy="0 0 0"/>
-        </joint>
-        <link name="tcp_gripper" />
-        <joint name="tool0-tcp_gripper" type="fixed">
-            <parent link="tool0"/>
-            <child link="tcp_gripper"/>
-            <origin xyz="0 0 $(arg tcp_offset)" rpy="0 0 $(arg tcp_z_rot)"/>
-        </joint>
     </xacro:if>
+    <link name="tcp_gripper" />
+    <joint name="tool0-tcp_gripper" type="fixed">
+        <parent link="tool0"/>
+        <child link="tcp_gripper"/>
+        <origin xyz="0 0 $(arg tcp_offset)" rpy="0 0 $(arg tcp_z_rot)"/>
+    </joint>
 </robot>

Commit message: Solved tf config mismatch within urdf and srdf

File: models/urdf/ur10e_eecam.urdf.xacro (robot description, xacro)
@@ -7,4 +7,5 @@
     <xacro:arg name="ur_type" default="ur10e"/>
     <xacro:arg name="tf_prefix" default=""/>
+    <xacro:arg name="parent_link" default="world_ur"/>
     <xacro:arg name="joint_limits_parameters_file" default="$(find ur_description)/config/$(arg ur_type)/joint_limits.yaml"/>
     <xacro:arg name="kinematics_parameters_file" default="$(find ur_description)/config/$(arg ur_type)/default_kinematics.yaml"/>
@@ -12,18 +13,25 @@
     <xacro:arg name="camera"                        default="true"/>
     <xacro:arg name="gripper"                       default="true"/>
-    <xacro:arg name="gfloor"                        default="true"/>
+    <xacro:arg name="gfloor"                        default="false"/>
     <xacro:arg name="gripper_collision_box"         default="false"/>
+    <xacro:arg name="back_wall"                     default="false"/>
     <xacro:arg name="tcp_offset"                    default="0.148"/>
     <xacro:arg name="tcp_z_rot"                     default="0.0"/>
+    <xacro:arg name="camera_pitch"                  default="0.41"/>
     <xacro:property name="camera"                   value="$(arg camera)"/>
     <xacro:property name="gripper"                  value="$(arg gripper)"/>
     <xacro:property name="gfloor"                   value="$(arg gfloor)"/>
+    <xacro:property name="back_wall"                value="$(arg back_wall)"/>
     <xacro:property name="gripper_collision_box"    value="$(arg gripper_collision_box)"/>
     <xacro:property name="tcp_offset"               value="$(arg tcp_offset)"/>
     <xacro:property name="tcp_z_rot"                value="$(arg tcp_z_rot)"/>
+    <xacro:property name="parent_link"              value="$(arg parent_link)"/>
+    <xacro:property name="camera_pitch"             value="$(arg camera_pitch)"/>
     <!-- Create the manipulator -->
-    <link name="world_ur"/>
+    <xacro:if value="${parent_link == 'world_ur'}">
+        <link name="world_ur"/>
+    </xacro:if>
     <xacro:ur_robot
-        parent="world_ur"
+        parent="${parent_link}"
         name="$(arg name)"
         tf_prefix="$(arg tf_prefix)"
@@ -42,4 +50,11 @@
         />
     </xacro:if>
+    <!-- TCP gripper inclusion -->
+    <link name="tcp_gripper" />
+    <joint name="tool0-tcp_gripper" type="fixed">
+        <parent link="tool0"/>
+        <child link="tcp_gripper"/>
+        <origin xyz="0 0 $(arg tcp_offset)" rpy="0 0 $(arg tcp_z_rot)"/>
+    </joint>
     <!-- Camera inclusion -->
     <xacro:if value="${camera}">
@@ -109,9 +124,3 @@
         </link>
     </xacro:if>
-    <link name="tcp_gripper" />
-    <joint name="tool0-tcp_gripper" type="fixed">
-        <parent link="tool0"/>
-        <child link="tcp_gripper"/>
-        <origin xyz="0 0 $(arg tcp_offset)" rpy="0 0 $(arg tcp_z_rot)"/>
-    </joint>
 </robot>

File: models/urdf/ur10e_mobile.urdf.xacro (robot description, xacro)
@@ -5,18 +5,18 @@
     <!-- Robot Arguments -->
     <xacro:arg name="name" default="ur"/>
-    <xacro:arg name="ur_type" default="ur5e"/>
+    <xacro:arg name="ur_type" default="ur10e"/>
     <xacro:arg name="tf_prefix" default=""/>
     <xacro:arg name="parent_link" default="world_ur"/>
-    <xacro:arg name="joint_limits_parameters_file" default="$(find ur_description)/config/ur5e/joint_limits.yaml"/>
-    <xacro:arg name="kinematics_parameters_file" default="$(find ur_description)/config/ur5e/default_kinematics.yaml"/>
+    <xacro:arg name="joint_limits_parameters_file" default="$(find ur_description)/config/$(arg ur_type)/joint_limits.yaml"/>
+    <xacro:arg name="kinematics_parameters_file" default="$(find ur_description)/config/$(arg ur_type)/default_kinematics.yaml"/>
     <!-- Additional objects Arguments -->
-    <xacro:arg name="camera"                        default="true"/>
-    <xacro:arg name="gripper"                       default="true"/>
+    <xacro:arg name="camera"                        default="false"/>
+    <xacro:arg name="gripper"                       default="false"/>
     <xacro:arg name="gfloor"                        default="false"/>
     <xacro:arg name="gripper_collision_box"         default="false"/>
     <xacro:arg name="back_wall"                     default="false"/>
-    <xacro:arg name="tcp_offset"                    default="0.148"/>
-    <xacro:arg name="tcp_z_rot"                     default="1.866"/>
-    <xacro:arg name="camera_pitch"                  default="0.41"/>
+    <xacro:arg name="tcp_offset"                    default="0.0"/>
+    <xacro:arg name="tcp_z_rot"                     default="0.0"/>
+    <xacro:arg name="camera_pitch"                  default="0.0"/>
     <xacro:property name="camera"                   value="$(arg camera)"/>
     <xacro:property name="gripper"                  value="$(arg gripper)"/>
@@ -38,6 +38,6 @@
         joint_limits_parameters_file="$(arg joint_limits_parameters_file)"
         kinematics_parameters_file="$(arg kinematics_parameters_file)"
-        physical_parameters_file="$(find ur_description)/config/ur5e/physical_parameters.yaml"
-        visual_parameters_file="$(find ur_description)/config/ur5e/visual_parameters.yaml"
+        physical_parameters_file="$(find ur_description)/config/$(arg ur_type)/physical_parameters.yaml"
+        visual_parameters_file="$(find ur_description)/config/$(arg ur_type)/visual_parameters.yaml"
     >
         <origin xyz="0 0 0" rpy="0 0 0" />
@@ -80,5 +80,5 @@
         <link name="floor">
             <visual> <!-- floor -->
-                <origin xyz="0.0 0.0 0.0" rpy="0 0 0"/>
+                <origin xyz="0.0 0.0 -0.40" rpy="0 0 0"/>
                 <geometry>
                     <box size="10 10 0.01"/>
@@ -89,8 +89,38 @@
             </visual>
             <collision>
-                <origin xyz="0.0 0.0 0.0" rpy="0 0 0"/>
+                <origin xyz="0.0 0.0 -0.40" rpy="0 0 0"/>
                 <geometry>
                     <box size="10 10 0.01"/>
                 </geometry>
+            </collision>
+            <visual>
+                <geometry>
+                    <box size="1.0 0.7 0.5"/> <!-- box sotto -->
+                </geometry>
+                <origin xyz="-0.25 0.0 -0.25" rpy="0 0 0"/>
+                <material name="">
+                        <color rgba="1.0 1.0 1.0 1.0"/>
+                </material>
+            </visual>
+            <visual>
+                <geometry>
+                    <box size="0.6 0.7 0.4"/> <!-- box sopra -->
+                </geometry>
+                <origin xyz="-0.4 0.0 0.2" rpy="0 0 0"/>
+                <material name="">
+                    <color rgba="1.0 1.0 1.0 1.0"/>
+                </material>
+            </visual>
+            <collision>
+                <geometry>
+                    <box size="1.0 0.7 0.5"/> <!-- box sotto -->
+                </geometry>
+                <origin xyz="-0.25 0.0 -0.25" rpy="0 0 0"/>
+            </collision>
+            <collision>
+                <geometry>
+                    <box size="0.6 0.7 0.4"/> <!-- box sopra -->
+                </geometry>
+                <origin xyz="-0.4 0.0 0.2" rpy="0 0 0"/>
             </collision>
         </link>
@@ -99,28 +129,4 @@
             <child link="floor"/>
             <origin xyz="0 0 -0.005" rpy="0 0 0"/>
-        </joint>
-    </xacro:if>
-    <xacro:if value="${back_wall}">
-        <link name="back_wall">
-            <visual> <!-- back wall -->
-                <origin xyz="-0.4 0 1.1" rpy="0 0 0"/>
-                <geometry>
-                    <box size="0.01 10 2.0"/>
-                </geometry>
-                <material name="">
-                    <color rgba="0.8 0.1 0.1 0.4"/>
-                </material>
-            </visual>
-            <collision>
-                <origin xyz="-0.4 0 1.1" rpy="0 0 0"/>
-                <geometry>
-                    <box size="0.01 10 2.0"/>
-                </geometry>
-            </collision>
-        </link>
-        <joint name="world_back_wall" type="fixed">
-            <parent link="base_link"/>
-            <child link="back_wall"/>
-            <origin xyz="0 0 0" rpy="0 0 0"/>
         </joint>
     </xacro:if>

File: models/urdf/ur5e_mobile.urdf.xacro (robot description, xacro)
@@ -7,23 +7,31 @@
     <xacro:arg name="ur_type" default="ur5e"/>
     <xacro:arg name="tf_prefix" default=""/>
+    <xacro:arg name="parent_link" default="world_ur"/>
     <xacro:arg name="joint_limits_parameters_file" default="$(find ur_description)/config/$(arg ur_type)/joint_limits.yaml"/>
     <xacro:arg name="kinematics_parameters_file" default="$(find ur_description)/config/$(arg ur_type)/default_kinematics.yaml"/>
     <!-- Additional objects Arguments -->
-    <xacro:arg name="camera"                        default="true"/>
-    <xacro:arg name="gripper"                       default="true"/>
-    <xacro:arg name="gfloor"                        default="true"/>
+    <xacro:arg name="camera"                        default="false"/>
+    <xacro:arg name="gripper"                       default="false"/>
+    <xacro:arg name="gfloor"                        default="false"/>
     <xacro:arg name="gripper_collision_box"         default="false"/>
-    <xacro:arg name="tcp_offset"                    default="0.148"/>
+    <xacro:arg name="back_wall"                     default="false"/>
+    <xacro:arg name="tcp_offset"                    default="0.0"/>
     <xacro:arg name="tcp_z_rot"                     default="0.0"/>
+    <xacro:arg name="camera_pitch"                  default="0.0"/>
     <xacro:property name="camera"                   value="$(arg camera)"/>
     <xacro:property name="gripper"                  value="$(arg gripper)"/>
     <xacro:property name="gfloor"                   value="$(arg gfloor)"/>
+    <xacro:property name="back_wall"                value="$(arg back_wall)"/>
     <xacro:property name="gripper_collision_box"    value="$(arg gripper_collision_box)"/>
     <xacro:property name="tcp_offset"               value="$(arg tcp_offset)"/>
     <xacro:property name="tcp_z_rot"                value="$(arg tcp_z_rot)"/>
+    <xacro:property name="parent_link"              value="$(arg parent_link)"/>
+    <xacro:property name="camera_pitch"             value="$(arg camera_pitch)"/>
     <!-- Create the manipulator -->
-    <link name="world_ur"/>
+    <xacro:if value="${parent_link == 'world_ur'}">
+        <link name="world_ur"/>
+    </xacro:if>
     <xacro:ur_robot
-        parent="world_ur"
+        parent="${parent_link}"
         name="$(arg name)"
         tf_prefix="$(arg tf_prefix)"
@@ -42,4 +50,11 @@
         />
     </xacro:if>
+    <!-- TCP gripper inclusion -->
+    <link name="tcp_gripper" />
+    <joint name="tool0-tcp_gripper" type="fixed">
+        <parent link="tool0"/>
+        <child link="tcp_gripper"/>
+        <origin xyz="0 0 $(arg tcp_offset)" rpy="0 0 $(arg tcp_z_rot)"/>
+    </joint>
     <!-- Camera inclusion -->
     <xacro:if value="${camera}">
@@ -141,9 +156,3 @@
         </link>
     </xacro:if>
-    <link name="tcp_gripper" />
-    <joint name="tool0-tcp_gripper" type="fixed">
-        <parent link="tool0"/>
-        <child link="tcp_gripper"/>
-        <origin xyz="0 0 $(arg tcp_offset)" rpy="0 0 $(arg tcp_z_rot)"/>
-    </joint>
 </robot>

File: models/urdf/ur_robotiq_85_gripper_macro.xacro (robot description, xacro)
@@ -12,13 +12,4 @@
             <origin xyz="0 0 0" rpy="0 -1.57 1.57" />
         </xacro:robotiq_85_gripper>
-        <!-- Create a non visual link to mark the tool center point -->
-        <link name="tcp_gripper">
-            <origin xyz="0 0 0" rpy="0 0 0" />
-        </link>
-        <joint name="tool0_to_tcp_joint" type="fixed">
-            <origin xyz="0 0 0.165" rpy="0 0 0" />
-            <parent link="${tf_prefix}tool0" />
-            <child link="tcp_gripper" />
-        </joint>
   </xacro:macro>
 </robot>
