Commit message: Cartesian plan and wait, routines devel

File: models/srdf/ur_floor.srdf.xacro (robot description, xacro)
@@ -9,3 +9,5 @@
     <!-- Disable collisions for Robotiq 85 gripper -->
     <disable_collisions link1="ee_collision_box" link2="wrist_3_link" reason="Adjacent" />
+    <!-- Disable collisions for camera -->
+    <disable_collisions link1="ee_collision_box" link2="camera_link" reason="Never" />
 </robot>

File: models/urdf/ur_floor.urdf.xacro (robot description, xacro)
@@ -18,3 +18,19 @@
     >
     </xacro:ur_floor>
+    <xacro:include filename="$(find realsense2_description)/urdf/_d435i.urdf.xacro"/>
+    <link name="d435i_base_link" />
+    <joint name="tool0-d4351_base_link" type="fixed">
+        <parent link="tool0"/>
+        <child link="d435i_base_link"/>
+        <origin xyz="0 -0.0775 0.024" rpy="0 -1.57 1.57"/>
+    </joint>
+    <link name="camera_detection_link" />
+    <joint name="camera_link-camera_detection_link" type="fixed">
+        <parent link="camera_link"/>
+        <child link="camera_detection_link"/>
+        <origin xyz="0 0 0" rpy="0 1.57 0"/>
+    </joint>
+    <xacro:sensor_d435i parent="d435i_base_link" name="camera">
+        <origin xyz="0 0 0" rpy="0 0 0" />
+    </xacro:sensor_d435i>
 </robot>
