Commit message: Modified joy and planning utilities

File: models/srdf/ur5e_robotiq_85_gripper.srdf.xacro (robot description, xacro)
@@ -18,4 +18,6 @@
         <link name="$(arg prefix)robotiq_85_right_inner_knuckle_link"/>
     </group>
+    <!-- Virtual base joint -->
+    <virtual_joint name="fixed_base" type="fixed" parent_frame="world" child_link="base_link" />
     <!-- Disable collisions for Robotiq 85 gripper -->
     <disable_collisions link1="$(arg prefix)robotiq_85_base_link" link2="wrist_3_link" reason="Adjacent" />

File: models/urdf/ur_robotiq_85_gripper_macro.xacro (robot description, xacro)
@@ -1,6 +1,9 @@
 <?xml version="1.0"?>
 <robot xmlns:xacro="http://ros.org/wiki/xacro">
+    <!-- Robot URDF file-->
     <xacro:include filename="$(find ur_description)/urdf/ur_macro.xacro"/>
+    <!-- Robotiq 85 Gripper URDF file -->
     <xacro:include filename="$(find robotiq_85_description)/urdf/robotiq_85_gripper_macro.urdf.xacro"/>
+    <!-- Gripper macro definition -->
     <xacro:macro name="ur_robotiq_85_gripper" params="
         robot_name
@@ -9,14 +12,15 @@
         joint_limits_parameters_file
         kinematics_parameters_file
-        ">
-        <!--This will create the gripper and attach it to the flange link -->
+        "
+    >
+        <!-- Create a link for the 'tool0' as parent for the gripper -->
         <xacro:robotiq_85_gripper
             prefix="${tf_prefix}"
-            parent="${tf_prefix}flange"
+            parent="${tf_prefix}tool0"
         >
-            <origin xyz="0 0 0" rpy="0 0 0" />
+            <origin xyz="0 0 0" rpy="0 -1.57 1.57" />
         </xacro:robotiq_85_gripper>
         <!-- Create a non visual link to mark the tool center point -->
-        <link name="tcp_link">
+        <link name="tcp_gripper">
             <origin xyz="0 0 0" rpy="0 0 0" />
         </link>
@@ -24,7 +28,8 @@
             <origin xyz="0 0 0.165" rpy="0 0 0" />
             <parent link="${tf_prefix}tool0" />
-            <child link="tcp_link" />
+            <child link="tcp_gripper" />
         </joint>
         <!--This will create the specific robot-->
+        <link name="world"/>
         <xacro:ur_robot
             parent="world"
