Commit message: Added xacro_args launch parameter, renamed end effector camera to 'ee_cam'

File: models/urdf/ur5e_robotiq_85_gripper.urdf.xacro (robot description, xacro)
@@ -10,10 +10,12 @@
     <xacro:arg name="kinematics_parameters_file" default="$(find ur_description)/config/$(arg ur_type)/default_kinematics.yaml"/>
     <!-- Additional objects Arguments -->
-    <xacro:arg name="camera"    default="true"/>
-    <xacro:arg name="gripper"   default="true"/>
-    <xacro:arg name="gfloor"    default="false"/>
-    <xacro:property name="camera"   value="$(arg camera)"/>
-    <xacro:property name="gripper"  value="$(arg gripper)"/>
-    <xacro:property name="gfloor"   value="$(arg gfloor)"/>
+    <xacro:arg name="camera"                   default="true"/>
+    <xacro:arg name="gripper"                  default="true"/>
+    <xacro:arg name="gfloor"                   default="false"/>
+    <xacro:arg name="gripper_collision_box"    default="false"/>
+    <xacro:property name="camera"                value="$(arg camera)"/>
+    <xacro:property name="gripper"               value="$(arg gripper)"/>
+    <xacro:property name="gfloor"                value="$(arg gfloor)"/>
+    <xacro:property name="gripper_collision_box" value="$(arg gripper_collision_box)"/>
     <!-- Create the manipulator -->
     <link name="world"/>
@@ -45,5 +47,5 @@
             <origin xyz="0 -0.0775 0.024" rpy="0 -1.57 1.57"/>
         </joint>
-        <xacro:sensor_d435i parent="d435i_base_link" name="camera">
+        <xacro:sensor_d435i parent="d435i_base_link" name="ee_cam">
             <origin xyz="0 0 0" rpy="0 0 0" />
         </xacro:sensor_d435i>
@@ -72,3 +74,32 @@
         </joint>
     </xacro:if>
+    <!-- Gripper collision box -->
+    <xacro:if value="${gripper_collision_box}">
+        <link name="ee_collision_box">
+            <visual>
+                <geometry>
+                    <box size="0.130 0.170 0.160"/>
+                </geometry>
+                <material name="">
+                    <color rgba="0.8 0.1 0.1 0.4"/>
+                </material>
+            </visual>
+            <collision>
+                <geometry>
+                    <box size="0.130 0.170 0.160"/>
+                </geometry>
+            </collision>
+        </link>
+        <joint name="tool0-ee_collision_box" type="fixed">
+            <parent link="tool0"/>
+            <child link="ee_collision_box"/>
+            <origin xyz="0 -0.04 0.080" rpy="0 0 0"/>
+        </joint>
+        <link name="tcp_gripper" />
+        <joint name="tool0-tcp_gripper" type="fixed">
+            <parent link="tool0"/>
+            <child link="tcp_gripper"/>
+            <origin xyz="0 0 0.145" rpy="0 0 0"/>
+        </joint>
+    </xacro:if>
 </robot>
