Commit message: Solved memory corruption issues in dynamic planner, MP might still need some revision

File: models/srdf/ur5e_eecam.srdf.xacro (robot description, xacro)
@@ -9,7 +9,7 @@
     <!-- Additional objects Arguments -->
     <xacro:arg name="camera"                   default="true"/>
-    <xacro:arg name="gripper"                  default="true"/>
-    <xacro:arg name="gfloor"                   default="false"/>
-    <xacro:arg name="gripper_collision_box"    default="false"/>
+    <xacro:arg name="gripper"                  default="false"/>
+    <xacro:arg name="gfloor"                   default="true"/>
+    <xacro:arg name="gripper_collision_box"    default="true"/>
     <xacro:property name="camera"                value="$(arg camera)"/>
     <xacro:property name="gripper"               value="$(arg gripper)"/>

File: models/urdf/ur5e_eecam.urdf.xacro (robot description, xacro)
@@ -13,9 +13,12 @@
     <xacro:arg name="gfloor"                        default="true"/>
     <xacro:arg name="gripper_collision_box"         default="true"/>
+    <xacro:arg name="back_wall"                     default="false"/>
     <xacro:arg name="tcp_offset"                    default="0.160"/>
-    <xacro:arg name="tcp_z_rot"                     default="0.300"/>
+    <xacro:arg name="tcp_z_rot"                     default="1.866"/>
+    <xacro:arg name="camera_pitch"                  default="0.0"/>
     <xacro:property name="camera"                   value="$(arg camera)"/>
     <xacro:property name="gripper"                  value="$(arg gripper)"/>
     <xacro:property name="gfloor"                   value="$(arg gfloor)"/>
+    <xacro:property name="back_wall"                value="$(arg back_wall)"/>
     <xacro:property name="gripper_collision_box"    value="$(arg gripper_collision_box)"/>
     <xacro:property name="tcp_offset"               value="$(arg tcp_offset)"/>
@@ -44,12 +47,18 @@
     <xacro:if value="${camera}">
         <xacro:include filename="$(find realsense2_description)/urdf/_d435i.urdf.xacro"/>
+        <link name="camera_mount" />
+        <joint name="tcp_gripper-camera_mount" type="fixed">
+            <parent link="tcp_gripper"/>
+            <child link="camera_mount"/>
+            <origin xyz="-0.070 0 -0.135" rpy="0 $(arg camera_pitch) 0"/>
+        </joint>
         <link name="d435i_base_link" />
-        <joint name="tool0-d435i_base_link" type="fixed">
-            <parent link="tool0"/>
+        <joint name="camera_mount-d435i_base_link" type="fixed">
+            <parent link="camera_mount"/>
             <child link="d435i_base_link"/>
-            <origin xyz="0 -0.0775 0.024" rpy="0 -1.57 1.57"/>
+            <origin xyz="0 0 0.021" rpy="0 0 0"/>
         </joint>
         <xacro:sensor_d435i parent="d435i_base_link" name="ee_cam">
-            <origin xyz="0 0 0" rpy="0 0 0" />
+            <origin xyz="0 0 0" rpy="0 -1.57 0" />
         </xacro:sensor_d435i>
     </xacro:if>
@@ -58,5 +67,5 @@
         <link name="floor">
             <visual> <!-- floor -->
-                <origin xyz="0.0 0.0 -0.40" rpy="0 0 0"/>
+                <origin xyz="0.0 0.0 0.0" rpy="0 0 0"/>
                 <geometry>
                     <box size="10 10 0.01"/>
@@ -67,5 +76,5 @@
             </visual>
             <collision>
-                <origin xyz="0.0 0.0 -0.40" rpy="0 0 0"/>
+                <origin xyz="0.0 0.0 0.0" rpy="0 0 0"/>
                 <geometry>
                     <box size="10 10 0.01"/>
@@ -77,4 +86,28 @@
             <child link="floor"/>
             <origin xyz="0 0 -0.005" rpy="0 0 0"/>
+        </joint>
+    </xacro:if>
+    <xacro:if value="${back_wall}">
+        <link name="back_wall">
+            <visual> <!-- back wall -->
+                <origin xyz="-0.4 0 1.1" rpy="0 0 0"/>
+                <geometry>
+                    <box size="0.01 10 2.0"/>
+                </geometry>
+                <material name="">
+                    <color rgba="0.8 0.1 0.1 0.4"/>
+                </material>
+            </visual>
+            <collision>
+                <origin xyz="-0.4 0 1.1" rpy="0 0 0"/>
+                <geometry>
+                    <box size="0.01 10 2.0"/>
+                </geometry>
+            </collision>
+        </link>
+        <joint name="world_back_wall" type="fixed">
+            <parent link="base_link"/>
+            <child link="back_wall"/>
+            <origin xyz="0 0 0" rpy="0 0 0"/>
         </joint>
     </xacro:if>
